Commit message: Editing has been made in the model.

File: src/simulation/models/urdf/marble_husky.urdf (robot description, URDF)
Before this commit: robot robot_name, 2 links, 1 joints
Links:
- link base_link: geometry collision box size=${base_length} ${base_width} ${base_height}; visual box size=${base_length} ${base_width} ${base_height}
