Commit message: urdf file model body and wheel parts complete

File: src/modules/vehicle_control_software/urdf/vehicle.urdf (robot description, URDF)
Before this commit: robot orion, 2 links, 1 joints
Links:
- added link left_back_wheel_link, mass 0.5; collision cylinder length=0.022 radius=0.033; visual mesh filename=package://vehicle_control_software/urdf/meshes/wheel.stl
- added link left_front_wheel_link, mass 0.5; collision cylinder length=0.022 radius=0.033; visual mesh filename=package://vehicle_control_software/urdf/meshes/wheel.stl
- added link right_back_wheel_link, mass 0.5; collision cylinder length=0.022 radius=0.033; visual mesh filename=package://vehicle_control_software/urdf/meshes/wheel.stl
- added link right_front_wheel_link, mass 0.5; collision cylinder length=0.022 radius=0.033; visual mesh filename=package://vehicle_control_software/urdf/meshes/wheel.stl
Joints:
- added joint wheel_left_back_joint: type continuous, parent base_link, child left_back_wheel_link, origin xyz=0.07 -0.08 0.033 rpy=1.57 0 0.0, axis 0 0 1
- added joint wheel_left_front_joint: type continuous, parent base_link, child left_front_wheel_link, origin xyz=-0.06 -0.08 0.033 rpy=1.57 0 0.0, axis 0 0 1
- added joint wheel_right_back_joint: type continuous, parent base_link, child right_back_wheel_link, origin xyz=0.07 0.08 0.033 rpy=-1.57 0 0.0, axis 0 0 1
- added joint wheel_right_front_joint: type continuous, parent base_link, child right_front_wheel_link, origin xyz=-0.06 0.08 0.033 rpy=-1.57 0 0.0, axis 0 0 1

Commit message: urdf file model body and wheel parts complete

File: src/modules/vehicle_control_software/urdf/vehicle.urdf (robot description, URDF)
Before this commit: robot orion, 6 links, 5 joints
Joints:
- removed joint wheel_left_back_joint
- removed joint wheel_left_front_joint
- removed joint wheel_right_back_joint
- removed joint wheel_right_front_joint
- added joint left_back_wheel_joint: type continuous, parent base_link, child left_back_wheel_link, origin xyz=-0.07 0.08 0.033 rpy=-1.57 0 0.0, axis 0 0 1
- added joint left_front_wheel_joint: type continuous, parent base_link, child left_front_wheel_link, origin xyz=0.06 0.08 0.033 rpy=-1.57 0 0.0, axis 0 0 1
- added joint right_back_wheel_joint: type continuous, parent base_link, child right_back_wheel_link, origin xyz=-0.07 -0.08 0.033 rpy=1.57 0 0.0, axis 0 0 1
- added joint right_front_wheel_joint: type continuous, parent base_link, child right_front_wheel_link, origin xyz=0.06 -0.08 0.033 rpy=1.57 0 0.0, axis 0 0 1

Commit message: Urdf file update

File: src/modules/vehicle_control_software/urdf/vehicle.urdf (robot description, URDF)
Before this commit: robot orion, 6 links, 5 joints
Links:
- added link front_camera_link; visual mesh filename=package://vehicle_control_software/urdf/meshes/rpi_camera.s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
- added link hc_sr04_left_link; visual mesh filename=package://vehicle_control_software/urdf/meshes/hc_sr04.stl
- added link hc_sr04_right_link; visual mesh filename=package://vehicle_control_software/urdf/meshes/hc_sr04.stl
Joints:
- added joint front_camera_joint: type fixed, parent base_link, child front_camera_link, origin xyz=0.09 0.0 0.048 rpy=1.55 0.0 1.57
- added joint hc_sr04_left_joint: type fixed, parent base_link, child hc_sr04_left_link, origin xyz=0.09 0.042 0.055 rpy=1.55 0.0 1.78
- added joint hc_sr04_right_joint: type fixed, parent base_link, child hc_sr04_right_link, origin xyz=0.09 -0.044 0.055 rpy=1.55 0.0 1.41
